File: 4. MCU data logger.kicad_pcb (KiCad board)
At the start: 2 copper layers, 29 parts, among them J1 Conn_01x04_Pin, J2 Conn_01x04_Pin, J3 Conn_01x09_Pin, J4 Conn_02x03_Odd_Even, U1 24LC1025, U2 24LC1025, U4 ATMEGA328P-AU, U5 DS1337S_, Y1 32.768 KHz, Y2 16 MHz

Commit message: components placed
Parts:
- moved J3 107.6 mm to (52.1, 87.6), turned to 90 degrees
- moved Y1 100.7 mm to (49.0, 79.6), turned to 90 degrees
- moved J2 90.8 mm to (78.1, 87.6), turned to 90 degrees
- moved C1 90.6 mm to (65.0, 61.5)
- moved C2 88.0 mm to (69.1, 61.5)
- moved U5 87.0 mm to (57.9, 78.7)
- moved U2 86.0 mm to (58.2, 62.9)
- moved BT1 85.8 mm to (48.9, 69.2)
- moved C3 85.5 mm to (73.3, 61.6)
- moved C5 85.2 mm to (74.4, 66.5)
- moved C4 83.4 mm to (77.5, 61.6)
- moved J4 82.6 mm to (87.0, 66.0)
- moved U1 82.4 mm to (58.0, 71.1)
- moved H1 82.3 mm to (47.6, 61.6)
- moved Y2 80.9 mm to (69.0, 82.9)
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Other:
- board outline added: 50.2 x 30.3 mm

Commit message: Routing Completed
Parts:
- moved C2 22.0 mm to (80.7, 80.2)
- moved C4 16.3 mm to (80.7, 77.6)
- moved R6 9.36 mm to (85.4, 65.4)
- moved C5 5.44 mm to (75.6, 61.3), turned to 180 degrees
- moved R5 4.08 mm to (85.4, 68.7)
- moved Y1 3.85 mm to (48.1, 75.9)
- moved H4 3.83 mm to (95.5, 89.7)
- moved R4 3.69 mm to (80.6, 72.2)
- moved H3 3.56 mm to (45.3, 89.7)
- moved H2 3.55 mm to (95.5, 59.3)
- moved BT1 3.50 mm to (48.2, 65.8)
- moved U4 3.28 mm to (70.4, 71.2)
- moved H1 3.27 mm to (45.3, 59.3)
- moved C3 3.21 mm to (70.2, 61.2)
- moved J4 3.17 mm to (90.2, 66.0)
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Routing:
- net /VCC: track 0.00 -> 175.4 mm, vias 0 -> 6
- net /SCK: track 0.00 -> 91.7 mm, vias 0 -> 3
- net GND: track 0.00 -> 81.6 mm, vias 0 -> 6
- net Net-(BT1-+): track 0.00 -> 73.0 mm, vias 0 -> 8
- net /SDA: track 0.00 -> 67.7 mm, vias 0 -> 8
- net /MISO: track 0.00 -> 33.9 mm, vias 0 -> 2
- net /D2: track 0.00 -> 32.9 mm
- net /RESET: track 0.00 -> 31.4 mm, vias 0 -> 2
- net Net-(U4-PB6): track 0.00 -> 29.3 mm, vias 0 -> 2
- net /RX: track 0.00 -> 28.5 mm, vias 0 -> 2
- net /D3: track 0.00 -> 27.8 mm
- net /TX: track 0.00 -> 27.6 mm, vias 0 -> 2
- net Net-(U4-PB7): track 0.00 -> 26.4 mm, vias 0 -> 2
- net /MOSI: track 0.00 -> 25.4 mm
- net /D4: track 0.00 -> 24.8 mm
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- added copper zone on F.Cu, net /VCC
- added copper zone on B.Cu, net GND
Other:
- board size 50.2 x 30.3 mm -> 55.8 x 35.9 mm

Commit message: Completed 2layer project
Parts:
- added REF**: KiCad-Logo2_5mm_SilkScreen, Symbol:KiCad-Logo2_5mm_SilkScreen, B.Cu at (56.9, 64.3)
Connections:
- BT1 pad 1: Net-(BT1-+) -> /VCC
- C2 pad 1: Net-(BT1-+) -> /VCC
- D2 pad 2: Net-(BT1-+) -> /VCC
- U4 pad 18: Net-(BT1-+) -> /VCC
- U4 pad 4: Net-(BT1-+) -> /VCC
Routing:
- net Net-(BT1-+): track 73.0 -> 0.00 mm, vias 8 -> 0
- net /VCC: track 175.4 -> 246.1 mm, vias 6 -> 14
- net GND: track 81.6 -> 71.1 mm, vias 6 -> 7
Other:
- board size 55.8 x 35.9 mm -> 55.4 x 35.4 mm
- board text added: "1"
- board text added: "2"
- board text added: "3"
- board text added: "4"
- board text added: "5"
- board text added: "6"
- board text added: "7"
- board text added: "GND"
- board text added: "GPIO"
- board text added: "I2C"
- board text added: "ICSP"
- board text added: "ICSP MISO|VCC SCK |MOSI RESET|GND"
- board text added: "MCU DATALOGGER"
- board text added: "RX"
- board text added: "SCK"
- board text added: "SDA"
- board text added: "SERIAL"
- board text added: "TX"
- board text added: "VCC"

Commit message: Fixed defects in schematic
Connections:
- J1 pad 4: /SCK -> /SCL
- R3 pad 2: /SCK -> /SCL
- U1 pad 6: /SCK -> /SCL
- U2 pad 6: /SCK -> /SCL
- U4 pad 28: /SCK -> /SCL
- U5 pad 6: /SCK -> /SCL
Routing:
- net /SCL: track 0.00 -> 76.9 mm, vias 0 -> 6
- net /SCK: track 91.8 -> 27.7 mm, vias 3 -> 2
- net /VCC: track 246.1 -> 230.2 mm, vias 14 -> 16
- net GND: track 71.1 -> 77.3 mm, vias 7 -> 8
- net Net-(U4-AREF): track 13.1 -> 14.0 mm
- net /SDA: track 67.7 -> 68.5 mm

Commit message: Fixed defects in pcb
Routing:
- net /VCC: track 230.2 -> 242.4 mm
Changed lines of the file:
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@@
+	)
+	(segment
+		(start 79.6074 68.8772)
+		(end 79.6074 68.6816)
+		(width 0.2)
+		(layer "F.Cu")
+		(net 2)
 	)
 	(segment
@@
 	)
 	(segment
+		(start 87.122 67.056)
+		(end 87.2254 66.9526)
+		(width 0.3)
+		(layer "F.Cu")
+		(net 2)
+	)
+	(segment
 		(start 51.562 63.6016)
 		(end 50.6984 64.4652)
@@
 	)
 	(segment
+		(start 87.2254 66.9526)
+		(end 87.2254 60.483932)
+		(width 0.3)
+		(layer "F.Cu")
+		(net 2)
+	)
+	(segment
 		(start 73.685978 73.0476)
 		(end 74.528 73.0476)
@@
 	)
 	(segment
+		(start 83.494 60.113)
+		(end 82.2914 61.3156)
+		(width 0.3)
+		(layer "F.Cu")
+		(net 2)
+	)
+	(segment
 		(start 64.14 61.468)
 		(end 64.394 61.214)
@@
 	)
 	(segment
+		(start 86.854468 60.113)
+		(end 83.494 60.113)
+		(width 0.3)
+		(layer "F.Cu")
+		(net 2)
+	)
+	(segment
 		(start 77.8256 72.5424)
 		(end 79.3534 72.5424)
@@
 	)
 	(segment
+		(start 74.528 73.2216)
+		(end 75.263 73.2216)
+		(width 0.2)
+		(layer "F.Cu")
+		(net 2)
+	)
+	(segment
 		(start 72.136 68.5292)
 		(end 72.136 70.612)
@@
 	)
 	(segment
-		(start 79.6074 68.8772)
-		(end 79.6074 68.6816)
-		(width 0.2)
-		(layer "F.Cu")
-		(net 2)
-	)
-	(segment
 		(start 90.688182 69.831)
 		(end 89.58952 69.831)
@@
 	)
 	(segment
-		(start 74.528 73.2216)
-		(end 75.263 73.2216)
-		(width 0.2)
-		(layer "F.Cu")
-		(net 2)
-	)
-	(segment
 		(start 75.946 74.676)
 		(end 75.9968 74.7268)
@@
 	)
 	(segment
+		(start 87.2254 60.483932)
+		(end 86.854468 60.113)
+		(width 0.3)
+		(layer "F.Cu")
+		(net 2)
+	)
+	(segment
 		(start 67.5132 70.093712)
 		(end 67.457256 70.149656)
@@
 		(layer "F.Cu")
 		(hatch edge 0.5)
+		(priority 1)
 		(connect_pads
 			(clearance 0.5)
@@
 		(polygon
 			(pts
-				(xy 48.260361 59.595342) (xy 92.862761 59.493742) (xy 93.573961 61.830542) (xy 95.047161 61.830542)
-				(xy 95.148761 86.519342) (xy 92.557961 88.398942) (xy 92.557961 89.465742) (xy 49.123961 89.313342)
-				(xy 45.923561 86.671742) (xy 45.872761 62.541742)
+				(xy 47.752 59.69) (xy 92.202 59.69) (xy 95.25 62.484) (xy 95.25 86.614) (xy 91.948 89.408) (xy 48.26 89.408)
+				(xy 45.974 86.868) (xy 45.974 61.976) (xy 47.498 60.96)
 			)
 		)
